File: pcb/exp-mmw-int/base/icyradio-exp-mmw-int-base.sch (EAGLE design)
At the start: 22 parts, among them U1 ATSAMD20E16A-M, U3 24AA02XX-X/OT

Commit message: pcb: Finish mmWave integrated expansion PCBs for production
Signed-off-by: João Silva <jgc3silva@gmail.com>
Parts:
- removed JP4, JP5: PINHD-2X3, Pin Header:PINHD-2X3
- removed JP8, JP9: PINHD-2X2, Pin Header:PINHD-2X2
- removed SJ1: (no value), Solder Jumper:SJ2CS
- added C10, C17, C18, C19, C20, C26, C27, C28, C29, C35, C36, C41, C42, C5: 1uF, Capacitor:CAPACITOR-0402
- added C12, C13, C21, C22, C23, C24, C37, C38, C6, C7, C9: 100nF, Capacitor:CAPACITOR-0402
- added C14: 1nF, Capacitor:CAPACITOR-0402
- added C15: 330pF, Capacitor:CAPACITOR-0402
- added C16, C34: 10uF, Capacitor:CAPACITOR-0603
- added C25, C39, C40: 10nF, Capacitor:CAPACITOR-0402
- added C30, C31, C32, C33, C43, C44: 10uF, Capacitor:CAPACITOR-0402
- added D1: LED0603, LED:LED0603
- added FB2: 1uH, Inductor:FERRITE-0603
- added JP1, JP3: PINHD-2X3, Pin Header:PINHD-2X3
- added P1, P10, P11, P12, P13, P14, P15, P16, P17, P18, P19, P2, P20, P21, P22, P23, P24, P25, P26, P27, P28, P29, P3, P30, P31, P32, P33, P34, P35, P36, P37, P38, P39, P4, P40, P41, P42, P43, P44, P45, P46, P47, P48, P49, P5, P50, P51, P52, P53, P54, P55, P56, P57, P58, P59, P6, P60, P61, P62, P63, P64, P65, P66, P67, P7, P8, P9: CHOLE-0.9MM-LAND, PADs:CHOLE-0.9MM-LAND
- added Q1, Q2: AO3400, Alpha Omega:AO3400
- added R10, R11, R14, R15, R16, R37, R38, R39, R40, R41, R8: 10K Ohms, Resistor:RESISTOR-0402
- added R12, R21, R35: DNP, Resistor:RESISTOR-0402
- added R13, R22, R36: 0 Ohms, Resistor:RESISTOR-0402
- added R17, R18, R19, R20, R23, R24, R25, R26, R27: 22 Ohms, Resistor:RESISTOR-0402
- added R2, R30, R31, R4: 4.7K Ohms, Resistor:RESISTOR-0402
- added R28, R29, R34, R5: 1K Ohms, Resistor:RESISTOR-0402
- added R32, R33: 2K Ohms, Resistor:RESISTOR-0402
- added U10, U11: ADM7171ACPZ-3.3, Analog Devices:ADM7171ACPZ-3.3
- added U2: FXL4TD245BQX, ON Semiconductor:FXL4TD245BQX
- added U4: MCP4728-A0, Microchip:MCP4728-A0
- added U5: MCP6V32-E/MNY, Microchip:MCP6V32-E/MNY
- added U6, U7: ADP7142AUJZ-1.8, Analog Devices:ADP7142AUJZ-1.8
- added U8: ADP7102ACPZ-1.5, Analog Devices:ADP7102ACPZ-1.5
- added U9: ADM7171ACPZ-5.0, Analog Devices:ADM7171ACPZ-5.0
- C11: value 100nF -> 10uF
- C2: value 10uF -> 1uF
- C8: value 1uF -> 100nF
- R6, R7: value 4.7K Ohms -> 10K Ohms
- U1: value ATSAMD20E16A-M -> ATSAMD21E18A-M; device Microchip:ATSAMD20E16A-M -> Microchip:ATSAMD21E18A-M
- U3: value 24AA02XX-X/OT -> FXL4TD245BQX; device Microchip:24AA02XX-X/OT -> ON Semiconductor:FXL4TD245BQX
Connections:
- net MCU_SWCLK renamed SWCLK
- net MCU_SWDIO renamed SWDIO
- removed net EE_I2C_SCL: JP8-4.S, U3.SCL
- removed net EE_I2C_SDA: JP8-2.S, U3.SDA
- removed net EE_WP: SJ1.2, U3.WP
- removed net EXT_IO_1_1: JP2-2.S, JP9-3.S, R3.1
- removed net EXT_IO_1_2: JP2-1.S, JP9-1.S, R1.1
- new net !RX_RST_1V8: P1.TP, Q1.D, R10.1
- new net !RX_SPI_CS: R16.1, R22.1, U1.PA28, U3.A0
- new net !RX_SPI_CS_1V8: R15.1, R17.2, U3.B0
- new net !RX_SPI_OE: R21.1, R22.2, U3.!OE
- new net !TX_RST_1V8: P35.TP, Q2.D, R14.1
- new net !TX_SPI_CS: R13.1, R9.1, U1.PA10, U2.A0
- new net !TX_SPI_CS_1V8: R23.2, R26.2, R7.1, U2.B0
- new net !TX_SPI_OE: R12.1, R13.2, U2.!OE
- new net 1V5_RF_RX: C28.C1, C32.C1, P57.TP, U8.SENSE, U8.VOUT
- new net 1V8_RF_RX: C27.C1, C31.C1, C8.C1, P58.TP, P59.TP, R10.2, R15.2, R36.2, U3.VCCB, U7.SENSE/ADJ, U7.VOUT
- new net 1V8_RF_TX: C26.C1, C30.C1, C6.C1, P49.TP, P50.TP, R14.2, R36.1, R7.2, U2.VCCB, U6.SENSE/ADJ, U6.VOUT
- new net 3V3_DAC_OPA: C11.C1, C12.C1, C13.C1, FB2.2, U4.VDD, U5.PWR.V+
- new net 3V3_RF_RX: C42.C1, C44.C1, P60.TP, P61.TP, P62.TP, P63.TP, P64.TP, P65.TP, U11.SENSE, U11.VOUT
- new net 3V3_RF_TX: C41.C1, C43.C1, P51.TP, P52.TP, P53.TP, P54.TP, P55.TP, P56.TP, U10.SENSE, U10.VOUT
- new net 5V0_RF_LO: C29.C1, C33.C1, P66.TP, P67.TP, U9.SENSE, U9.VOUT
- new net DAC_I2C_SCL: R1.1, U1.PA09, U4.SCL
- new net DAC_I2C_SDA: R2.1, U1.PA08, U4.SDA
- new net LED: D1.A, U1.PA11
- new net LO_ANA_PWR_EN: R37.2, U1.PA00, U9.EN
- new net N$10: P5.TP, R20.1
- new net N$11: P37.TP, R26.1
- new net N$12: P36.TP, R23.1
- new net N$13: P38.TP, R24.1
- new net N$14: P39.TP, R27.1
- new net N$15: P40.TP, R25.1
- new net N$16: D1.C, R5.2
- new net N$2: C40.C1, U11.SS
- new net N$3: C25.C1, U9.SS
- new net N$4: R28.1, R31.2, U5.1.-IN
- new net N$5: R29.1, R30.2, U5.1.+IN
- new net N$6: R32.2, U5.2.-IN, U5.2.OUT
- new net N$7: P2.TP, R17.1
- new net N$8: P3.TP, R19.1
- new net N$9: P4.TP, R18.1
- new net N$96: C39.C1, U10.SS
- new net RF_SPI_MISO: U1.PA05, U2.A3, U3.A3
- new net RF_SPI_MOSI: U1.PA06, U2.A2, U3.A2
- new net RF_SPI_SCK: U1.PA07, U2.A1, U3.A1
- new net RX_ANA_PWR_EN: R38.2, U1.PA19, U11.EN, U8.EN/UVLO
- new net RX_DIG_PWR_EN: R40.2, U1.PA22, U7.EN
- new net RX_GAIN_VCTRL: P44.TP, U4.VOUTA
- new net RX_PWR_VDET: P43.TP, U5.2.+IN
- new net RX_PWR_VDET_DIV: C14.C1, R32.1, R34.2, U1.PA03
- new net RX_RST: Q1.G, R8.2, U1.PA27
- new net RX_SPI_MISO_1V8: R18.2, U3.B3
- new net RX_SPI_MOSI_1V8: R20.2, U3.B2
- new net RX_SPI_SCK_1V8: R19.2, U3.B1
- new net TX_ANA_PWR_EN: R39.2, U1.PA01, U10.EN
- new net TX_DIG_PWR_EN: R41.2, U1.PA23, U6.EN
- new net TX_GAIN_VCTRL1: P45.TP, U4.VOUTD
- new net TX_GAIN_VCTRL2: P46.TP, U4.VOUTC
- new net TX_PWR_VDET: R31.1, R33.2, U5.1.OUT
- new net TX_PWR_VDET_DIV: C15.C1, R33.1, R35.2, U1.PA02
- new net TX_PWR_VDET_N: P48.TP, R28.2
- new net TX_PWR_VDET_P: P47.TP, R29.2
- new net TX_RST: Q2.G, R11.2, U1.PA04
- new net TX_SPI_MISO_1V8: R27.2, U2.B3
- new net TX_SPI_MOSI_1V8: R25.2, U2.B2
- new net TX_SPI_SCK_1V8: R24.2, U2.B1
- net !MCU_RESET: now also R6.1; no longer R9.1
- net 2V5: now also JP3-2.S; no longer JP4-2.S
- net 3V3: now also C10.C1, C16.C1, C17.C1, C18.C1, C19.C1, C21.C1, C22.C1, C23.C1, C7.C1, C9.C1, FB2.1, JP3-1.S, R16.2, R2.2, R4.2, U2.T/!R!0, U2.T/!R!1, U2.T/!R!2, U2.VCCA, U3.T/!R!0, U3.T/!R!1, U3.T/!R!2, U3.VCCA, U6.VIN, U7.VIN, U8.VIN; no longer C11.C1, JP4-1.S, R7.2, SJ1.3, U3.VCC
- net 5V0: now also C20.C1, C24.C1, C34.C1, C35.C1, C36.C1, C37.C1, C38.C1, JP3-5.S, JP3-6.S, U10.VIN, U11.VIN, U9.VIN; no longer JP4-5.S, JP4-6.S
- net EXT_CLK_2_3: now also JP2-3.S; no longer JP5-3.S
- net EXT_IO_1_3: now also JP1-4.S, U1.PA14; no longer JP2-4.S
- net EXT_IO_1_4: now also JP1-3.S, U1.PA15; no longer JP2-3.S
- net EXT_IO_1_5: now also JP1-6.S, U1.PA25; no longer JP2-6.S
- net EXT_IO_2_2: now also JP2-6.S; no longer JP5-6.S
- net EXT_IO_2_4: now also JP2-4.S; no longer JP5-4.S
- net EXT_IO_2_6: now also JP2-2.S; no longer JP5-2.S
- net GND: now also C10.C2, C12.C2, C13.C2, C14.C2, C15.C2, C16.C2, C17.C2, C18.C2, C19.C2, C20.C2, C21.C2, C22.C2, C23.C2, C24.C2, C25.C2, C26.C2, C27.C2, C28.C2, C29.C2, C30.C2, C31.C2, C32.C2, C33.C2, C34.C2, C35.C2, C36.C2, C37.C2, C38.C2, C39.C2, C40.C2, C41.C2, C42.C2, C43.C2, C44.C2, C5.C2, C6.C2, C7.C2, C9.C2, JP1-5.S, JP2-1.S, JP3-3.S, JP3-4.S, P10.TP, P11.TP, P12.TP, P13.TP, P14.TP, P15.TP, P16.TP, P17.TP, P18.TP, P19.TP, P20.TP, P21.TP, P22.TP, P23.TP, P24.TP, P25.TP, P26.TP, P27.TP, P28.TP, P29.TP, P30.TP, P31.TP, P32.TP, P33.TP, P34.TP, P41.TP, P42.TP, P6.TP, P7.TP, P8.TP, P9.TP, Q1.S, Q2.S, R11.1, R12.2, R21.2, R30.1, R34.1, R35.1, R37.1, R38.1, R39.1, R40.1, R41.1, R5.1, R8.1, U10.GND, U11.GND, U2.GND, U2.T/!R!3, U3.GND, U3.T/!R!3, U4.!LDAC, U4.VSS, U5.PWR.V-, U6.GND, U7.GND, U8.GND, U9.GND; no longer JP4-3.S, JP4-4.S, JP5-1.S, JP5-5.S, SJ1.1, U3.VSS
- net MCU_I2C_SCL: now also JP1-2.S, R3.1; no longer JP9-4.S, R6.1
- net MCU_I2C_SDA: now also JP1-1.S, R4.1; no longer JP9-2.S, R7.1
- net N$1: now also C5.C1; no longer C8.C1
Other:
- note added: "(VDET - GND) -> 0 mV to 1034 mV (ADC Vref = 1100 mV)"
- note added: "(VDET_P - VDET_N) -> 0 mV to 220 mV"
- note added: "0 mV to 1100 mV (ADC Vref = 1100 mV)"
- note added: "0 mV to 3300 mV"
- note added: "0 mV to 3300 mV (Buffered)"
- note added: "Compat. w/ ADP150"
- note added: "DNP if RX digital 1V8 reg. is installed"
- note added: "DNP if TX digital 1V8 reg. is used for RX digital 1V8"
- note added: "EXT_CLK_2_3"
- note added: "EXT_IO_1_1"
- note added: "EXT_IO_1_2"
- note added: "EXT_IO_1_3"
- note added: "EXT_IO_1_4"
- note added: "EXT_IO_1_5"
- note added: "EXT_IO_2_2"
- note added: "EXT_IO_2_4"
- note added: "EXT_IO_2_6"
- note added: "LPF fc = 240 kHz approx."
- note added: "Place only one resistor"
- note added: "Range is 0 mV to 1800 mV (DAC Vref = 2048 mV)"
