File: pcb/exp-mmw-int/rf/icyradio-exp-mmw-int-rf.sch (EAGLE design)
At the start: 68 parts, among them U1 ADMV1013, U2 ADMV1014

Commit message: pcb: Finish mmWave integrated expansion PCBs for production
Signed-off-by: João Silva <jgc3silva@gmail.com>
Parts:
- added C55, C60: 5.6pF, Capacitor:CAPACITOR-0402
- added C56, C61: 18pF, Capacitor:CAPACITOR-0402
- added C57, C62: 1nF, Capacitor:CAPACITOR-0402
- added C58, C63: 100nF, Capacitor:CAPACITOR-0402
- added C59: 10uF, Capacitor:CAPACITOR-0402
- added L1: DNP, Inductor:INDUCTOR-0402
- added L2, L3: 3.3nH, Inductor:INDUCTOR-0402
- added P1, P10, P2, P22, P23, P24, P25, P26, P27, P28, P29, P3, P33, P34, P35, P36, P37, P38, P39, P4, P5, P52, P53, P54, P55, P56, P57, P58, P59, P6, P60, P64, P65, P7, P8, P9: CHOLE-0.9MM-SS, PADs:CHOLE-0.9MM-SS
- added P11, P12, P13, P14, P15, P16, P17, P18, P19, P20, P21, P30, P31, P32, P40, P41, P42, P43, P44, P45, P46, P47, P48, P49, P50, P51, P61, P62, P63, P66, P67: CHOLE-0.9MM-DS, PADs:CHOLE-0.9MM-DS
- added R10, R13, R18: 0 Ohms, Resistor:RESISTOR-0402
- added R11, R12, R14, R15, R16, R17, R19, R20: DNP, Resistor:RESISTOR-0402
- added R21, R22, R23: 16.7 Ohms, Resistor:RESISTOR-0402
- added R8: 1.1K Ohms, Resistor:RESISTOR-0402
- added R9: 50 Ohms, Resistor:RESISTOR-0402
- added RFCON5: RFCON-U.FL, RF Connector:RFCON-U.FL
- added U3: ADMV1013, Analog Devices:ADMV1013
- added U4: BFCV-2895+, Mini Circuits:BFCV-2895+
- added U5: QCN-34+, Mini Circuits:QCN-34+
- added U6: ADMV1014, Analog Devices:ADMV1014
- added U7, U8: AVA-183A+, Mini Circuits:AVA-183A+
- C11, C23, C26, C32, C41, C50, C53: value 10nF -> 100pF
- C13, C25, C31, C40, C52: value 10uF -> 100pF
- C15, C27, C33, C42, C45, C54, C6: value 100pF -> 10uF
- C17, C35, C44, C5: value 10nF -> 10uF
- C19, C22, C37, C46, C49, C7: value 10uF -> 10nF
- C21, C30, C36, C48, C9: value 100pF -> 10nF
- R1: value 0 Ohms -> 50 Ohms
- R2, R4: value 0 Ohms -> 1K Ohms
- R3: value 0 Ohms -> 1.1K Ohms
- R6, R7: value 1.1K Ohms -> 50 Ohms
- RFCON2, RFCON4: value RFCON-U.FL -> RFCON-HK-R-SR2-SA; device RF Connector:RFCON-U.FL -> RF Connector:RFCON-HK-R-SR2-SA
- U1: value ADMV1013 -> BFCV-2895+; device Analog Devices:ADMV1013 -> Mini Circuits:BFCV-2895+
- U2: value ADMV1014 -> QCN-34+; device Analog Devices:ADMV1014 -> Mini Circuits:QCN-34+
Connections:
- removed net N$1: R1.2, RFCON1.SIGNAL
- removed net N$2: R2.2, RFCON2.SIGNAL
- removed net N$3: R3.2, RFCON3.SIGNAL
- removed net N$4: R4.2, RFCON4.SIGNAL
- removed net N$7: U1.IF_I
- removed net N$8: U1.IF_Q
- removed net TX_BB_I_N: R2.1, U1.I_N
- removed net TX_BB_I_P: R1.1, U1.I_P
- removed net TX_BB_Q_N: R4.1, U1.Q_N
- removed net TX_BB_Q_P: R3.1, U1.Q_P
- new net 5V0_RF_LO: C54.C1, C55.C1, C56.C1, C57.C1, C59.C1, C60.C1, C61.C1, C62.C1, L2.1, L3.1, P64.TP, P65.TP, U7.VD2, U8.VD2
- new net LO_AMP1_IN: L1.1, R10.1, U7.RFIN
- new net LO_AMP1_OUT: R11.2, R12.2, R13.2, U7.RFOUT
- new net LO_AMP2_IN: R13.1, R14.2, R15.2, U8.RFIN
- new net LO_AMP2_OUT: R16.2, R17.2, R18.2, U8.RFOUT
- new net LO_AMP_VD1: C58.C1, L2.2, U7.VD1
- new net LO_AMP_VD2: C63.C1, L3.2, U8.VD1
- new net LO_IN: R10.2, RFCON5.SIGNAL
- new net LO_OUT: R18.1, R19.2, R20.2, R21.2
- new net LO_SPLIT: R21.1, R22.2, R23.2
- new net N$11: R1.2, U2.ISO
- new net N$13: R7.2, U5.ISO
- new net N$17: R2.2, U3.VCTRL1
- new net N$18: R4.2, U3.VCTRL2
- new net RX_GAIN_VCTRL: P34.TP, U6.VCTRL
- new net RX_IF: U4.RFIN, U5.SUM
- new net RX_IF_FILT: RFCON3.SIGNAL, U4.RFOUT
- new net RX_IF_I: U5.P90DEG, U6.IF_I
- new net RX_IF_Q: U5.0DEG, U6.IF_Q
- new net RX_LO: R22.1, U6.LO_P
- new net RX_LO_N: R9.2, U6.LO_N
- new net RX_PWR_VDET: P33.TP, U6.VDET
- new net RX_RF: RFCON4.SIGNAL, U6.RF_IN
- new net TX_GAIN_VCTRL1: P1.TP, R2.1
- new net TX_GAIN_VCTRL2: P2.TP, R4.1
- new net TX_IF_FILT: U1.RFOUT, U2.SUM
- new net TX_IF_I: U2.0DEG, U3.IF_I
- new net TX_IF_IN: RFCON1.SIGNAL, U1.RFIN
- new net TX_IF_Q: U2.P90DEG, U3.IF_Q
- new net TX_LO: R23.1, U3.LOP
- new net TX_LO_N: R6.2, U3.LON
- new net TX_PWR_VDET_N: P4.TP, U3.VENV_N
- new net TX_PWR_VDET_P: P3.TP, U3.VENV_P
- new net TX_RF: RFCON2.SIGNAL, U3.RF
- net !RX_RST: now also P39.TP, U6.RST; no longer U2.RST
- net !RX_SPI_SEN: now also P35.TP, U6.!SEN; no longer U2.!SEN
- net !TX_RST: now also P10.TP, U3.RST; no longer U1.RST
- net !TX_SPI_SEN: now also P6.TP, U3.!SEN; no longer U1.!SEN
- net !TX_SPI_SEN2: now also P5.TP, U3.!SEN2; no longer U1.!SEN2
- net 1V5_RF_RX: now also C45.C1, C49.C1, P52.TP, U6.VCC_LNA_1P5; no longer C52.C1, C54.C1, U2.VCC_LNA_1P5
- net 1V8_RF_RX: now also C33.C1, C36.C1, C39.C1, C42.C1, C46.C1, C50.C1, P53.TP, P54.TP, U6.DVDD, U6.VCC_VVA; no longer C16.C1, C17.C1, C18.C1, C28.C1, C29.C1, C30.C1, U2.DVDD, U2.VCC_VVA
- net 1V8_RF_TX: now also C11.C1, C15.C1, C19.C1, C23.C1, C7.C1, P22.TP, P23.TP, U3.DVDD, U3.VCC_VVA; no longer C1.C1, C2.C1, C3.C1, C5.C1, C6.C1, U1.DVDD, U1.VCC_VVA
- net 3V3_RF_RX: now also C27.C1, C28.C1, C29.C1, C30.C1, C31.C1, C32.C1, C51.C1, C52.C1, P55.TP, P56.TP, P57.TP, P58.TP, P59.TP, P60.TP, U6.VCC_BG, U6.VCC_IF_BB, U6.VCC_LNA_3P3, U6.VCC_MIXER, U6.VCC_QUAD, U6.VCC_VGA; no longer C36.C1, C39.C1, C42.C1, C45.C1, C46.C1, U2.VCC_BG, U2.VCC_IF_BB, U2.VCC_LNA_3P3, U2.VCC_MIXER, U2.VCC_QUAD, U2.VCC_VGA
- net 3V3_RF_TX: now also C1.C1, C16.C1, C17.C1, C18.C1, C2.C1, C3.C1, C5.C1, C6.C1, P24.TP, P25.TP, P26.TP, P27.TP, P28.TP, P29.TP, U3.VCC2_DRV, U3.VCC_AMP1, U3.VCC_AMP2, U3.VCC_BG, U3.VCC_BG2, U3.VCC_DRV, U3.VCC_ENV, U3.VCC_MIXER, U3.VCC_QUAD; no longer C11.C1, C15.C1, C19.C1, C23.C1, C27.C1, C31.C1, C32.C1, C33.C1, C7.C1, U1.VCC2_DRV, U1.VCC_AMP1, U1.VCC_AMP2, U1.VCC_BG, U1.VCC_BG2, U1.VCC_DRV, U1.VCC_ENV, U1.VCC_MIXER, U1.VCC_QUAD
- net GND: now also C55.C2, C56.C2, C57.C2, C58.C2, C59.C2, C60.C2, C61.C2, C62.C2, C63.C2, L1.2, P11.TP, P12.TP, P13.TP, P14.TP, P15.TP, P16.TP, P17.TP, P18.TP, P19.TP, P20.TP, P21.TP, P30.TP, P31.TP, P32.TP, P40.TP, P41.TP, P42.TP, P43.TP, P44.TP, P45.TP, P46.TP, P47.TP, P48.TP, P49.TP, P50.TP, P51.TP, P61.TP, P62.TP, P63.TP, P66.TP, P67.TP, R1.1, R11.1, R12.1, R14.1, R15.1, R16.1, R17.1, R19.1, R20.1, R3.1, R8.1, R9.1, RFCON5.GND, U3.GND, U4.GND, U5.GND, U6.GND, U7.GND, U8.GND
- net N$5: now also R3.2, U3.BG_RBIAS2; no longer R5.2, U1.BG_RBIAS2
- net N$6: now also R5.2, U3.BG_RBIAS1; no longer R6.2, U1.BG_RBIAS1
- net N$9: now also R8.2, U6.BG_RBIAS; no longer R7.2, U2.BG_RBIAS
- net RX_SPI_SCLK: now also P36.TP, U6.SCLK; no longer U2.SCLK
- net RX_SPI_SDI: now also P38.TP, U6.SDI; no longer U2.SDI
- net RX_SPI_SDO: now also P37.TP, U6.SDO; no longer U2.SDO
- net TX_SPI_SCLK: now also P7.TP, U3.SCLK; no longer U1.SCLK
- net TX_SPI_SDI: now also P9.TP, U3.SDI; no longer U1.SDI
- net TX_SPI_SDO: now also P8.TP, U3.SDO; no longer U1.SDO
Other:
- note added: "0 V (min. gain) to 1.8 V (max. gain)"
- note added: "0.6 V (low power) to 3.3 V (high power)"
- note added: "1.8 V (min. gain) to 0 V (max. gain)"
- note added: "Diff: 0 mV (low power) to 250 mV (high power) CM: TBD ??"
- note added: "LO AMP 1 (+12 dB to +15 dB)"
- note added: "LO AMP 2 (+12 dB to +15 dB)"
- note added: "Optional Attenuator"
- note added: "Optional match to get higher power from synth"
- note added: "Power divider (-6 dB)"
- note added: "VCC_BG + VCC_MIXER + VCC_QUAD"
- note removed: "VCC_BG + VCC_MIXER"
