File: pcb/exp-mmw-int/icyradio-exp-mmw-int.brd (EAGLE design)
At the start: 85.7 x 98.4 mm, 309 parts, among them Q1 AO3400, Q2 AO3400, U1 EFM32GG11B420F2048GQ64, U10 BFCV-2895+, U11 QCN-34+, U12 ADMV1013, U13 BFCV-2895+, U14 QCN-34+, U15 ADMV1014, U16 PMA2-123LN+, U17 ADRF5720, U18 PMA2-123LN+, U19 LTC5597, U2 MCP9802-A0, U20 ADRF5019, U21 ADRF5019, U22 LTC5597, U23 ADRF5019, U24 ADRF5019, U25 8V97003, U26 ADP7142AUJZ-3.3, U27 ADM7170ACPZ-5.0, U28 ADM7172ACPZ-3.3, U29 ADM8828, U3 MCP9802-A1, U30 ADP7142AUJZ-1.8, U31 ADP7142AUJZ-1.8, U32 ADP7102ACPZ-1.5, U33 ADM7171ACPZ-3.3, U34 ADM7171ACPZ-3.3, U4 MCP9802-A3, U5 FXL4TD245BQX, U6 FXL4TD245BQX, U7 MCP6V32-E/MNY, U8 MCP4728-A0, U9 MCP6V32-E/MNY

Commit message: pcb: Minor mmWave board schematic changes
Signed-off-by: João Silva <jgc3silva@gmail.com>
Parts:
- R12, R21: value 0 Ohms -> DNP
- R13, R22: value DNP -> 0 Ohms
Changed lines of the file:
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@@
 <drawing>
 <settings>
-<setting alwaysvectorfont="yes"/>
+<setting alwaysvectorfont="no"/>
 <setting verticaltext="up"/>
 </settings>
@@
 <attribute name="TOLERANCE" value="" x="62.8" y="25.4" size="1.778" layer="27" rot="R180" display="off"/>
 </element>
-<element name="R22" library="Resistor" package="RES0402" value="DNP" x="59.5" y="25.9" smashed="yes" rot="R180">
+<element name="R22" library="Resistor" package="RES0402" value="0 Ohms" x="59.5" y="25.9" smashed="yes" rot="R180">
 <attribute name="NAME" x="60.5" y="25.9" size="0.8" layer="25" font="vector" ratio="10" rot="SR0" align="center-left"/>
 <attribute name="POWER" value="" x="59.5" y="25.9" size="1.778" layer="27" rot="R180" display="off"/>
 <attribute name="TOLERANCE" value="" x="63.5" y="24.9" size="1.778" layer="27" rot="R180" display="off"/>
 </element>
-<element name="R21" library="Resistor" package="RES0402" value="0 Ohms" x="59.5" y="26.9" smashed="yes">
+<element name="R21" library="Resistor" package="RES0402" value="DNP" x="59.5" y="26.9" smashed="yes">
 <attribute name="NAME" x="60.5" y="26.9" size="0.8" layer="25" font="vector" ratio="10" rot="SR0" align="center-left"/>
 <attribute name="POWER" value="" x="59.5" y="26.9" size="1.778" layer="27" display="off"/>
@@
 <attribute name="NAME" x="47.4004" y="46" size="0.8" layer="25" font="vector" ratio="10" rot="SR0" align="center-left"/>
 <attribute name="POWER" value="" x="46.2996" y="46" size="1.778" layer="27" rot="R180" display="off"/>
+<attribute name="SERIES" value="FC0402" x="46.2996" y="46" size="1.778" layer="27" rot="R180" display="off"/>
 <attribute name="TOLERANCE" value="" x="65.2996" y="76" size="1.778" layer="27" rot="R180" display="off"/>
 </element>
@@
 <attribute name="NAME" x="35.2996" y="46" size="0.8" layer="25" font="vector" ratio="10" rot="SR0" align="center-left"/>
 <attribute name="POWER" value="" x="38.2996" y="46" size="1.778" layer="27" display="off"/>
+<attribute name="SERIES" value="FC0402" x="38.2996" y="46" size="1.778" layer="27" display="off"/>
 <attribute name="TOLERANCE" value="" x="24.2996" y="12" size="1.778" layer="27" display="off"/>
 </element>
@@
 <attribute name="VOLTAGE" value="" x="31.9794375" y="26.9" size="1.778" layer="27" rot="R180" display="off"/>
 </element>
-<element name="R13" library="Resistor" package="RES0402" value="DNP" x="47.9" y="22.5" smashed="yes" rot="R270">
+<element name="R13" library="Resistor" package="RES0402" value="0 Ohms" x="47.9" y="22.5" smashed="yes" rot="R270">
 <attribute name="NAME" x="47.9" y="23.5" size="0.8" layer="25" font="vector" ratio="10" rot="SR90" align="center-left"/>
 <attribute name="POWER" value="" x="48.2" y="22.7" size="1.778" layer="27" rot="R270" display="off"/>
 <attribute name="TOLERANCE" value="" x="48.2" y="22.7" size="1.778" layer="27" rot="R270" display="off"/>
 </element>
-<element name="R12" library="Resistor" package="RES0402" value="0 Ohms" x="46.9" y="22.5" smashed="yes" rot="R90">
+<element name="R12" library="Resistor" package="RES0402" value="DNP" x="46.9" y="22.5" smashed="yes" rot="R90">
 <attribute name="NAME" x="46.9" y="23.5" size="0.8" layer="25" font="vector" ratio="10" rot="SR90" align="center-left"/>
 <attribute name="POWER" value="" x="46.6" y="22.3" size="1.778" layer="27" rot="R90" display="off"/>
