File: pcb/main/icyradio-main.brd (EAGLE design)
At the start: 167.7 x 111.2 mm, 702 parts, among them CON101 FPC-22P, CON102 FPC-22P, CON1101 2EDG-2P-5MM-H, CON701 4P-SH-TOP, CON801 PCIE-X4-EDGE, J101 RJ45_MAG_LED_1G-TE-1-2301994-0, J701 TRSJACK, J702 TRSJACK, J703 TRSJACK, M701 SPH0641LM4H-1, M702 SPH0641LM4H-1, Q101 AO3400, Q102 AO3400, Q1101 AO3400, Q1102 AO4805, Q1103 AO3400, Q1104 AO4805, Q1105 AO4805, Q1106 AO3400, T501 UWB1-85E, T502 UWB1-85E, T503 UWB1-85E, T504 UWB1-85E, T505 UWB1-85E, T506 UWB1-85E, T507 UWB1-85E, T508 UWB1-85E, U1001 LTC4313-3, U1002 UPD301C, U1003 MIC2019, U101 MIC2019, U102 RPI-CM4, U1101 MCP1804-3302, U1102 LT7182S, U1201 ADM7172ACPZ-5.0, U1202 ADM7171ACPZ-1.3, U1203 ADM7171ACPZ-3.3, U1204 MIC23159, U1205 MIC5166, U1206 ADM7171ACPZ-1.3, U1207 ADM7171ACPZ-3.3, U1208 MIC23159, U1209 MIC23155, U1210 ADP7142AUJZ-3.3, U201 XC7A100TFGG484, U202 SST26VF064B, U301 MT41K256M16TW-125, U401 AD9361, U501 MIC2019, U502 MIC2019, U503 MIC2019, U504 MIC2019, U505 ADL5601, U506 ADL5601, U601 8V97003, U701 ADAU1372, U901 DSB321SDA, U902 SI5351C-B-GM

Commit message: pcb: Update 3V3 switching regulator inductor to 4.7 uH so it exits DCM pcb: Update transceiver clock DC-block capacitor to 100nF
Signed-off-by: João Silva <jgc3silva@gmail.com>
Parts:
- C403: value 10pF -> 100nF
- L1201, L1202, L1203, L1205: device Coilcraft:XGL351X -> Coilcraft:XGL35XX
- L1204: value 2.2uH -> 4.7uH; device Coilcraft:XGL351X -> Coilcraft:XGL35XX

Commit message: pcb: Change mmWave Synth loop filter component values
Signed-off-by: João Silva <jgc3silva@gmail.com>
Parts:
- C616: value 220nF -> 1uF
- C617: value 2.2nF -> 10nF
- C618: value 680pF -> 2.2nF
- R608: value 62 Ohms -> 20 Ohms
- R609: value 20 Ohms -> 62 Ohms
Changed lines of the file:
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@@
 <attribute name="VOLTAGE" value="" x="-1361.8" y="82.5" size="1.778" layer="27" rot="R270" display="off"/>
 </element>
-<element name="R608" library="Resistor" package="RES0402" value="62 Ohms" x="40.5" y="80.6" smashed="yes" rot="R90">
+<element name="R608" library="Resistor" package="RES0402" value="20 Ohms" x="40.5" y="80.6" smashed="yes" rot="R90">
 <attribute name="NAME" x="45.2" y="80.8" size="0.8" layer="25" font="vector" ratio="10" rot="SR270" align="center-left"/>
 <attribute name="POWER" value="" x="1437" y="80.6" size="1.778" layer="27" rot="R90" display="off"/>
 <attribute name="TOLERANCE" value="" x="1437" y="80.6" size="1.778" layer="27" rot="R90" display="off"/>
 </element>
-<element name="C616" library="Capacitor" package="CAP0402" value="220nF" x="40" y="79.1" smashed="yes" rot="R180">
+<element name="C616" library="Capacitor" package="CAP0402" value="1uF" x="40" y="79.1" smashed="yes" rot="R180">
 <attribute name="NAME" x="41" y="79.1" size="0.8" layer="25" font="vector" ratio="10" rot="SR0" align="center-left"/>
 <attribute name="VOLTAGE" value="" x="40" y="1478.1" size="1.778" layer="27" rot="R180" display="off"/>
 </element>
-<element name="R609" library="Resistor" package="RES0402" value="20 Ohms" x="38" y="81.1" smashed="yes">
+<element name="R609" library="Resistor" package="RES0402" value="62 Ohms" x="38" y="81.1" smashed="yes">
 <attribute name="NAME" x="37" y="82" size="0.8" layer="25" font="vector" ratio="10" rot="SR0" align="center-left"/>
 <attribute name="POWER" value="" x="38" y="-1320.4" size="1.778" layer="27" display="off"/>
 <attribute name="TOLERANCE" value="" x="38" y="-1320.4" size="1.778" layer="27" display="off"/>
 </element>
-<element name="C617" library="Capacitor" package="CAP0402" value="2.2nF" x="39.5" y="80.6" smashed="yes" rot="R270">
+<element name="C617" library="Capacitor" package="CAP0402" value="10nF" x="39.5" y="80.6" smashed="yes" rot="R270">
 <attribute name="NAME" x="44.2" y="80.8" size="0.8" layer="25" font="vector" ratio="10" rot="SR270" align="center-left"/>
 <attribute name="VOLTAGE" value="" x="-1364.5" y="80.6" size="1.778" layer="27" rot="R270" display="off"/>
 </element>
-<element name="C618" library="Capacitor" package="CAP0402" value="680pF" x="38" y="80.1" smashed="yes">
+<element name="C618" library="Capacitor" package="CAP0402" value="2.2nF" x="38" y="80.1" smashed="yes">
 <attribute name="NAME" x="36.4" y="79.1" size="0.8" layer="25" font="vector" ratio="10" rot="SR0" align="center-left"/>
 <attribute name="VOLTAGE" value="" x="38" y="-1326.4" size="1.778" layer="27" display="off"/>

Commit message: pcb: Update TCXO AC couple capacitor to 100nF
Signed-off-by: João Silva <jgc3silva@gmail.com>
Parts:
- C907: value 10pF -> 100nF
Changed lines of the file:
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@@
 <attribute name="VOLTAGE" value="" x="201.62" y="131.74" size="1.778" layer="27" rot="R90" display="off"/>
 </element>
-<element name="C907" library="Capacitor" package="CAP0402" value="10pF" x="65" y="14.9" smashed="yes" rot="R90">
+<element name="C907" library="Capacitor" package="CAP0402" value="100nF" x="65" y="14.9" smashed="yes" rot="R90">
 <attribute name="NAME" x="65" y="13.9" size="0.8" layer="25" font="vector" ratio="10" rot="SR270" align="center-left"/>
 <attribute name="VOLTAGE" value="" x="199.62" y="136.82" size="1.778" layer="27" rot="R90" display="off"/>

Commit message: Add new 8V97003 datasheet Add cooling fan expansion card (WIP) Updated some schematic resistors from 49.9R to 50R Sync mmWave expansion card firmware after some lab testing (WIP) Sync PMC firmware Sync RV firmware (WIP) Sync misc SoapySDR library work
Signed-off-by: João Silva <jgc3silva@gmail.com>
Parts:
- C623, C624, C625, C626: value 20pF -> 10nF
- R610, R611, R612, R613, R614, R615: value 49.9 Ohms -> 50 Ohms
Changed lines of the file:
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@@
 <attribute name="VOLTAGE" value="" x="37.4" y="92.4" size="1.778" layer="27" rot="R90" display="off"/>
 </element>
-<element name="R611" library="Resistor" package="RES0402" value="49.9 Ohms" x="30.7" y="85.5" smashed="yes" rot="R90">
+<element name="R611" library="Resistor" package="RES0402" value="50 Ohms" x="30.7" y="85.5" smashed="yes" rot="R90">
 <attribute name="POWER" value="" x="30.7" y="85.5" size="1.778" layer="27" rot="R90" display="off"/>
+<attribute name="SERIES" value="FC0402" x="30.7" y="85.5" size="1.778" layer="27" rot="R90" display="off"/>
 <attribute name="TOLERANCE" value="" x="30.7" y="85.5" size="1.778" layer="27" rot="R90" display="off"/>
 </element>
-<element name="R613" library="Resistor" package="RES0402" value="49.9 Ohms" x="30.7" y="83.5" smashed="yes" rot="R270">
+<element name="R613" library="Resistor" package="RES0402" value="50 Ohms" x="30.7" y="83.5" smashed="yes" rot="R270">
 <attribute name="NAME" x="29.7" y="82.4" size="0.8" layer="25" font="vector" ratio="10" rot="SR270" align="center-left"/>
 <attribute name="POWER" value="" x="31" y="83.6" size="1.778" layer="27" rot="R270" display="off"/>
+<attribute name="SERIES" value="FC0402" x="30.7" y="83.5" size="1.778" layer="27" rot="R270" display="off"/>
 <attribute name="TOLERANCE" value="" x="31" y="83.6" size="1.778" layer="27" rot="R270" display="off"/>
 </element>
@@
 <attribute name="VOLTAGE" value="" x="43.9" y="-1279.3" size="1.778" layer="27" display="off"/>
 </element>
-<element name="C626" library="Capacitor" package="CAP0402" value="20pF" x="29.2" y="85" smashed="yes" rot="R180">
+<element name="C626" library="Capacitor" package="CAP0402" value="10nF" x="29.2" y="85" smashed="yes" rot="R180">
 <attribute name="NAME" x="25.3" y="84" size="0.8" layer="25" font="vector" ratio="10" rot="SR0" align="center-left"/>
+<attribute name="SERIES" value="ATC520L" x="29.2" y="85" size="1.778" layer="27" rot="R180" display="off"/>
 <attribute name="VOLTAGE" value="" x="29.7" y="1452" size="1.778" layer="27" rot="R180" display="off"/>
 </element>
-<element name="C624" library="Capacitor" package="CAP0402" value="20pF" x="29.2" y="84" smashed="yes" rot="R180">
+<element name="C624" library="Capacitor" package="CAP0402" value="10nF" x="29.2" y="84" smashed="yes" rot="R180">
 <attribute name="NAME" x="25.3" y="83" size="0.8" layer="25" font="vector" ratio="10" rot="SR0" align="center-left"/>
+<attribute name="SERIES" value="ATC520L" x="29.2" y="84" size="1.778" layer="27" rot="R180" display="off"/>
 <attribute name="VOLTAGE" value="" x="29.7" y="1453.5" size="1.778" layer="27" rot="R180" display="off"/>
 </element>
-<element name="R615" library="Resistor" package="RES0402" value="49.9 Ohms" x="28.7" y="82.5" smashed="yes" rot="R90">
+<element name="R615" library="Resistor" package="RES0402" value="50 Ohms" x="28.7" y="82.5" smashed="yes" rot="R90">
 <attribute name="NAME" x="27.7" y="82.4" size="0.8" layer="25" font="vector" ratio="10" rot="SR270" align="center-left"/>
 <attribute name="POWER" value="" x="1400.7" y="82" size="1.778" layer="27" rot="R90" display="off"/>
+<attribute name="SERIES" value="FC0402" x="28.7" y="82.5" size="1.778" layer="27" rot="R90" display="off"/>
 <attribute name="TOLERANCE" value="" x="1400.7" y="82" size="1.778" layer="27" rot="R90" display="off"/>
 </element>
-<element name="C625" library="Capacitor" package="CAP0402" value="20pF" x="29.2" y="88" smashed="yes" rot="R180">
+<element name="C625" library="Capacitor" package="CAP0402" value="10nF" x="29.2" y="88" smashed="yes" rot="R180">
 <attribute name="NAME" x="25.5" y="89.1" size="0.8" layer="25" font="vector" ratio="10" rot="SR0" align="center-left"/>
+<attribute name="SERIES" value="ATC520L" x="29.2" y="88" size="1.778" layer="27" rot="R180" display="off"/>
 <attribute name="VOLTAGE" value="" x="29.7" y="1462.5" size="1.778" layer="27" rot="R180" display="off"/>
 </element>
-<element name="R614" library="Resistor" package="RES0402" value="49.9 Ohms" x="28.7" y="90.5" smashed="yes" rot="R270">
+<element name="R614" library="Resistor" package="RES0402" value="50 Ohms" x="28.7" y="90.5" smashed="yes" rot="R270">
 <attribute name="NAME" x="28.7" y="91.5" size="0.8" layer="25" font="vector" ratio="10" rot="SR90" align="center-left"/>
 <attribute name="POWER" value="" x="-1350.3" y="91" size="1.778" layer="27" rot="R270" display="off"/>
+<attribute name="SERIES" value="FC0402" x="28.7" y="90.5" size="1.778" layer="27" rot="R270" display="off"/>
 <attribute name="TOLERANCE" value="" x="-1350.3" y="91" size="1.778" layer="27" rot="R270" display="off"/>
 </element>
-<element name="C623" library="Capacitor" package="CAP0402" value="20pF" x="29.2" y="89" smashed="yes" rot="R180">
+<element name="C623" library="Capacitor" package="CAP0402" value="10nF" x="29.2" y="89" smashed="yes" rot="R180">
 <attribute name="NAME" x="25.5" y="90" size="0.8" layer="25" font="vector" ratio="10" rot="SR0" align="center-left"/>
+<attribute name="SERIES" value="ATC520L" x="29.2" y="89" size="1.778" layer="27" rot="R180" display="off"/>
 <attribute name="VOLTAGE" value="" x="29.7" y="1468.5" size="1.778" layer="27" rot="R180" display="off"/>
 </element>
-<element name="R610" library="Resistor" package="RES0402" value="49.9 Ohms" x="30.7" y="87.5" smashed="yes" rot="R270">
+<element name="R610" library="Resistor" package="RES0402" value="50 Ohms" x="30.7" y="87.5" smashed="yes" rot="R270">
 <attribute name="POWER" value="" x="-1353.8" y="88" size="1.778" layer="27" rot="R270" display="off"/>
+<attribute name="SERIES" value="FC0402" x="30.7" y="87.5" size="1.778" layer="27" rot="R270" display="off"/>
 <attribute name="TOLERANCE" value="" x="-1353.8" y="88" size="1.778" layer="27" rot="R270" display="off"/>
 </element>
-<element name="R612" library="Resistor" package="RES0402" value="49.9 Ohms" x="30.7" y="89.5" smashed="yes" rot="R90">
+<element name="R612" library="Resistor" package="RES0402" value="50 Ohms" x="30.7" y="89.5" smashed="yes" rot="R90">
 <attribute name="NAME" x="30.7" y="90.5" size="0.8" layer="25" font="vector" ratio="10" rot="SR90" align="center-left"/>
 <attribute name="POWER" value="" x="1414.7" y="89" size="1.778" layer="27" rot="R90" display="off"/>
+<attribute name="SERIES" value="FC0402" x="30.7" y="89.5" size="1.778" layer="27" rot="R90" display="off"/>
 <attribute name="TOLERANCE" value="" x="1414.7" y="89" size="1.778" layer="27" rot="R90" display="off"/>
 </element>
@@
 <element name="C619" library="Capacitor" package="CAP0402" value="10nF" x="31.7" y="90.5" smashed="yes" rot="R90">
 <attribute name="NAME" x="31.7" y="91.5" size="0.8" layer="25" font="vector" ratio="10" rot="SR90" align="center-left"/>
+<attribute name="SERIES" value="ATC520L" x="31.7" y="90.5" size="1.778" layer="27" rot="R90" display="off"/>
 <attribute name="VOLTAGE" value="" x="1420.7" y="90.5" size="1.778" layer="27" rot="R90" display="off"/>
 </element>
@@
 <element name="C620" library="Capacitor" package="CAP0402" value="10nF" x="31.7" y="82.5" smashed="yes" rot="R270">
 <attribute name="NAME" x="30.6" y="82.4" size="0.8" layer="25" font="vector" ratio="10" rot="SR270" align="center-left"/>
+<attribute name="SERIES" value="ATC520L" x="31.7" y="82.5" size="1.778" layer="27" rot="R270" display="off"/>
 <attribute name="VOLTAGE" value="" x="-1361.8" y="82.5" size="1.778" layer="27" rot="R270" display="off"/>
 </element>
